File: rc2014-icecore.sch (KiCad schematic (older format))
At the start: 21 parts, among them J1 Conn_01x39, J2 Conn_01x10, J3 Conn_02x15_Odd_Even, J4 Conn_02x13_Odd_Even, U1 LM1117-3.3, U2 SN74CB3T3245, U3 SN74CB3T3245, U4 SN74CB3T3245, U5 SN74CB3T3245, U6 SN74CB3T3245

Commit message: WIP of level shifter
Parts:
- removed A1: BE-CARRIER, blackedge:BE-CARRIER-SMD, symbol blackedge:BE-CARRIER
- removed H1: MountingHole, MountingHole:MountingHole_3.2mm_M3, symbol Mechanical:MountingHole
- removed J3: Conn_02x15_Odd_Even, Connector_PinSocket_2.54mm:PinSocket_2x15_P2.54mm_Horizontal, symbol Connector_Generic:Conn_02x15_Odd_Even
- removed J4: Conn_02x13_Odd_Even, Connector_PinHeader_2.54mm:PinHeader_2x13_P2.54mm_Horizontal, symbol Connector_Generic:Conn_02x13_Odd_Even
- added J3: Conn_02x25_Odd_Even, Connector_PinSocket_2.54mm:PinSocket_2x25_P2.54mm_Vertical, symbol Connector_Generic:Conn_02x25_Odd_Even
- added JP2: Jumper, Connector_PinHeader_2.54mm:PinHeader_1x02_P2.54mm_Vertical, symbol Device:Jumper
Connections:
- net labels removed: +3V3, AN5, AN6, AN7, AN8, AN9, EMISO, EMOSI, ESCK, P32, P33, P34, P35, P36, P37, P38, P39, P40, P41, P42, P43, P44, P45, P46, P47, RX, SCL, SDA, SWCLK, SWDIO, TCK, TDI, TDO, TMS, TX, ~ESS, ~RESET
- wire segments 309 -> 206
- no-connect marks 28 -> 6

Commit message: Rev 1 as sent to JLCPCB
Connections:
- wire segments 206 -> 207
- no-connect marks 6 -> 12
Changed lines of the file:
@@
 	530  3860 580  3860
 Wire Wire Line
-	12020 2350 12020 2550
+	12020 2350 12020 2470
 $Comp
 L power:+3.3V #PWR01
@@
 5V
 $Comp
-L power:GND #PWR?
+L power:GND #PWR0103
 U 1 1 6082819A
 P 3470 5290
-F 0 "#PWR?" H 3470 5040 50  0001 C CNN
+F 0 "#PWR0103" H 3470 5040 50  0001 C CNN
 F 1 "GND" V 3475 5162 50  0000 R CNN
 F 2 "" H 3470 5290 50  0001 C CNN
@@
 $EndComp
 $Comp
-L power:GND #PWR?
+L power:GND #PWR0104
 U 1 1 60828769
 P 3470 5390
-F 0 "#PWR?" H 3470 5140 50  0001 C CNN
+F 0 "#PWR0104" H 3470 5140 50  0001 C CNN
 F 1 "GND" V 3475 5262 50  0000 R CNN
 F 2 "" H 3470 5390 50  0001 C CNN
@@
 $EndComp
 $Comp
-L power:GND #PWR?
+L power:GND #PWR0105
 U 1 1 6083B5F6
 P 4470 5390
-F 0 "#PWR?" H 4470 5140 50  0001 C CNN
+F 0 "#PWR0105" H 4470 5140 50  0001 C CNN
 F 1 "GND" V 4475 5262 50  0000 R CNN
 F 2 "" H 4470 5390 50  0001 C CNN
@@
 $EndComp
 $Comp
-L power:GND #PWR?
+L power:GND #PWR0106
 U 1 1 6083BAD6
 P 4470 5290
-F 0 "#PWR?" H 4470 5040 50  0001 C CNN
+F 0 "#PWR0106" H 4470 5040 50  0001 C CNN
 F 1 "GND" V 4475 5162 50  0000 R CNN
 F 2 "" H 4470 5290 50  0001 C CNN
@@
 	0    -1   -1   0
 $EndComp
+NoConn ~ 870  5560
+NoConn ~ 870  5660
+NoConn ~ 870  5760
+NoConn ~ 870  5860
+NoConn ~ 870  5960
+$Comp
+L power:PWR_FLAG #FLG0101
+U 1 1 60A81E8E
+P 630 3760
+F 0 "#FLG0101" H 630 3835 50  0001 C CNN
+F 1 "PWR_FLAG" H 630 3933 50  0000 C CNN
+F 2 "" H 630 3760 50  0001 C CNN
+F 3 "~" H 630 3760 50  0001 C CNN
+	1    630  3760
+	1    0    0    -1
+$EndComp
+NoConn ~ 7240 4210
+$Comp
+L power:PWR_FLAG #FLG0102
+U 1 1 60A98D9F
+P 12020 2470
+F 0 "#FLG0102" H 12020 2545 50  0001 C CNN
+F 1 "PWR_FLAG" V 12020 2598 50  0000 L CNN
+F 2 "" H 12020 2470 50  0001 C CNN
+F 3 "~" H 12020 2470 50  0001 C CNN
+	1    12020 2470
+	0    1    1    0
+$EndComp
+Connection ~ 12020 2470
+Wire Wire Line
+	12020 2470 12020 2550
 $EndSCHEMATC
